Commit message: using our arm xacro file

File: catkin_ws/src/me212arm/model/my_robot.xacro (robot description, xacro)
@@ -1,5 +1,4 @@
-<!-- my_robot 2.12 Team 4a -->
-<?xml version="1.0">
-<robot name="my_robot">
+<?xml version="1.0"?>
+<robot xmlns:xacro="http://www.ros.org/wiki/xacro" name="my_robot">
 	<link name="base">
 		<visual>
@@ -37,9 +36,10 @@
 			</geometry>
 		</visual>
+	</link>
 	<joint name ="base_to_arm" type="prismatic">
 		<parent link="base"/>
 		<child link="arm"/>
 		<axis xyz="0 1 0"/>
-		<limit lower="-0.19" upper="0"/>
+		<limit effort="1" lower="-0.19" upper="0" velocity="1"/>
 		<origin xyz="-0.035 -0.105 -0.015"/>
 	</joint>
@@ -53,5 +53,5 @@
 		<child link="end_effector_1"/>
 		<axis xyz="0 1 0"/>
-		<limit lower="0" upper="1.58"/>
+		<limit effort="1" lower="0" upper="1.58" velocity="1"/>
 		<origin xyz="0.012 0.129 0.011"/>   <!-- UPDATE WITH CAD -->
 	</joint>
@@ -61,2 +61,3 @@
 		<origin xyz="0 -0.1085 0.04"/>
 	</joint>
+</robot>

Commit message: updated xacro file

File: catkin_ws/src/me212arm/model/my_robot.xacro (robot description, xacro)
@@ -1,8 +1,24 @@
 <?xml version="1.0"?>
 <robot xmlns:xacro="http://www.ros.org/wiki/xacro" name="my_robot">
-	<link name="base">
+<xacro:property name="base_l" value="0.07"/>
+<xacro:property name="base_w" value="0.06"/>
+<xacro:property name="base_h" value="0.04"/>
+<xacro:property name="arm_l" value="0.26"/>
+<xacro:property name="arm_w" value="0.01"/>
+<xacro:property name="arm_h" value="0.01"/>
+<xacro:property name="mount_l" value="0.50"/>
+<xacro:property name="mount_w" value="0.061"/>
+<xacro:property name="mount_h" value="0.07"/>
+<xacro:property name="end_effector_1_l" value="0.207"/>
+<xacro:property name="end_effector_1_w" value="0.01"/>
+<xacro:property name="end_effector_1_h" value="0.01"/>
+<xacro:property name="end_effector_2_l" value="0.01"/>
+<xacro:property name="end_effector_2_w" value="0.01"/>
+<xacro:property name="end_effector_2_h" value="0.08"/>
+<xacro:property name="pi" value="3.141592654"/>
+	<link name="base">   <!-- need to change x to y, y to -x -->
 		<visual>
 			<geometry>
-				<box size="0.06 0.07 0.04"/>
+				<box size="${base_l} ${base_w} ${base_h}"/>
 			</geometry>
 			<origin rpy="0 0 0" xyz="0 0 0"/> <!-- CHANGE LATER -->
@@ -12,6 +28,7 @@
 		<visual>
 			<geometry>
-				<box size="0.01 0.26 0.01"/>
+				<box size="${arm_l} ${arm_w} ${arm_h}"/>
 			</geometry>
+			<origin rpy="0 0 0" xyz="${(arm_length-base_length)/2} "/>
 		</visual>
 	</link>
@@ -19,6 +36,7 @@
 		<visual>
 			<geometry>
-				<box size="0.061 0.050 0.07"/>
+				<box size="${mount_l} ${mount_w} ${mount_h}"/>
 			</geometry>
+			<origin xyz=""/>
 		</visual>
 	</link>
@@ -26,6 +44,7 @@
 		<visual>
 			<geometry>
-				<box size="0.01 0.207 0.01"/>
+				<box size="${end_effector_1_l} ${end_effector_1_w} ${end_effector_1_h}"/>
 			</geometry>
+			<origin xyz=""/>
 		</visual>
 	</link>
@@ -33,6 +52,7 @@
 		<visual>
 			<geometry>
-				<box size="0.01 0.01 0.08"/>
+				<box size="${end_effector_2_l} ${end_effector_2_w} ${end_effector_2_h}"/>
 			</geometry>
+			<origin xyz=""/>
 		</visual>
 	</link>
@@ -42,10 +62,10 @@
 		<axis xyz="0 1 0"/>
 		<limit effort="1" lower="-0.19" upper="0" velocity="1"/>
-		<origin xyz="-0.035 -0.105 -0.015"/>
+		<origin xyz="${((base_l-arm_l)/2) + 0.028} ${-(base_w+arm_w)/2} ${(arm_h-base_h)/2}"/>
 	</joint>
 	<joint name ="arm_to_mount" type="fixed">
 		<parent link="arm"/>
 		<child link="mount"/>
-		<origin xyz="0.02 -0.155 0"/>
+		<origin xyz="${(arm_l+mount_l)/2} 0.02 0"/>
 	</joint>
 	<joint name ="mount_to_end_effector_1" type="revolute">
@@ -54,10 +74,10 @@
 		<axis xyz="0 1 0"/>
 		<limit effort="1" lower="0" upper="1.58" velocity="1"/>
-		<origin xyz="0.012 0.129 0.011"/>   <!-- UPDATE WITH CAD -->
+		<origin xyz="${(mount_l+end_effector_1_l)/2} 0.012 0.008"/>
 	</joint>
 	<joint name ="end_effector_1_to_end_effector_2" type="fixed">
 		<parent link="end_effector_1"/>
 		<child link="end_effector_2"/>
-		<origin xyz="0 -0.1085 0.04"/>
+		<origin xyz="${(end_effector_1_l-end_effector_2_l)/2} 0 ${(end_effector_2_h-end_effector_1_h)/2}"/>
 	</joint>
 </robot>
