Commit message: replacing me212arm xacro

File: catkin_ws/src/me212arm/model/me212arm.xacro (robot description, xacro)
@@ -1,69 +1,83 @@
 <?xml version="1.0"?>
-<robot xmlns:xacro="http://www.ros.org/wiki/xacro" name="me212bot">
-<xacro:property name="link1_length" value="0.1778" />
-<xacro:property name="link2_length" value="0.235" />
-<xacro:property name="M_PI" value="3.1415926" />
-<link name="arm_base">
-    <visual>
-        <geometry>
-            <box size="0.01 0.01 0.05" />
-        </geometry>
-        <origin rpy="0 0 0" xyz="0 0 0"/>
-        <material name="color1">
-            <color rgba="0.5 0.5 0.0 1"/>
-        </material>
-    </visual>
-</link>
-<link name="link1">
-    <visual>
-        <geometry>
-            <box size="0.01 0.01 ${link1_length}" />
-        </geometry>
-        <origin rpy="0 0 0" xyz="0 0 ${link1_length/2}"/>
-        <material name="color2">
-            <color rgba="0.5 0.0 0.5 1"/>
-        </material>
-    </visual>
-</link>
-<link name="link2">
-    <visual>
-        <geometry>
-            <box size="0.01 0.01 ${link2_length}" />
-        </geometry>
-        <origin rpy="0 0 0" xyz="0 0 ${link2_length/2}"/>
-        <material name="color3">
-            <color rgba="0.0 0.5 0.5 1"/>
-        </material>
-    </visual>
-</link>
-<link name="tcp">
-    <visual>
-        <geometry>
-            <sphere radius="0.01" />
-        </geometry>
-        <origin rpy="0 0 0" xyz="0 0 0"/>
-        <material name="color4">
-            <color rgba="0.5 0.5 0.5 1"/>
-        </material>
-    </visual>
-</link>
-<joint name="joint1" type="revolute">
-    <parent link="arm_base"/>
-    <child link="link1"/>
-    <origin xyz="0 0 0" />
-    <limit effort="300" lower="${-M_PI}" upper="${M_PI}" velocity="7.33"/>
-    <axis xyz="0 -1 0"/>
-</joint>
-<joint name="joint2" type="revolute">
-    <parent link="link1"/>
-    <child link="link2"/>
-    <origin xyz="0 0 ${link1_length}" />
-    <limit effort="300" lower="${-M_PI}" upper="${M_PI}" velocity="7.33"/>
-    <axis xyz="0 -1 0"/>
-</joint>
-<joint name="joint3" type="fixed">
-    <parent link="link2"/>
-    <child link="tcp"/>
-    <origin xyz="0 0 ${link2_length}" />
-</joint>
+<robot xmlns:xacro="http://www.ros.org/wiki/xacro" name="my_robot">
+<xacro:property name="base_l" value="0.07"/>
+<xacro:property name="base_w" value="0.06"/>
+<xacro:property name="base_h" value="0.04"/>
+<xacro:property name="arm_l" value="0.26"/>
+<xacro:property name="arm_w" value="0.01"/>
+<xacro:property name="arm_h" value="0.01"/>
+<xacro:property name="mount_l" value="0.50"/>
+<xacro:property name="mount_w" value="0.061"/>
+<xacro:property name="mount_h" value="0.07"/>
+<xacro:property name="end_effector_1_l" value="0.207"/>
+<xacro:property name="end_effector_1_w" value="0.01"/>
+<xacro:property name="end_effector_1_h" value="0.01"/>
+<xacro:property name="end_effector_2_l" value="0.01"/>
+<xacro:property name="end_effector_2_w" value="0.01"/>
+<xacro:property name="end_effector_2_h" value="0.08"/>
+<xacro:property name="pi" value="3.141592654"/>
+	<link name="base">
+		<visual>
+			<geometry>
+				<box size="${base_l} ${base_w} ${base_h}"/>
+			</geometry>
+			<origin rpy="0 0 0" xyz="0 0 0"/>
+		</visual>
+	</link>
+	<link name="arm">
+		<visual>
+			<geometry>
+				<box size="${arm_l} ${arm_w} ${arm_h}"/>
+			</geometry>
+			<origin rpy="0 0 0" xyz="${(arm_l-base_l)/2} "/>
+		</visual>
+	</link>
+	<link name="mount">
+		<visual>
+			<geometry>
+				<box size="${mount_l} ${mount_w} ${mount_h}"/>
+			</geometry>
+			<origin xyz=""/>
+		</visual>
+	</link>
+	<link name="end_effector_1">
+		<visual>
+			<geometry>
+				<box size="${end_effector_1_l} ${end_effector_1_w} ${end_effector_1_h}"/>
+			</geometry>
+			<origin xyz=""/>
+		</visual>
+	</link>
+	<link name="end_effector_2">
+		<visual>
+			<geometry>
+				<box size="${end_effector_2_l} ${end_effector_2_w} ${end_effector_2_h}"/>
+			</geometry>
+			<origin xyz=""/>
+		</visual>
+	</link>
+	<joint name ="base_to_arm" type="prismatic">
+		<parent link="base"/>
+		<child link="arm"/>
+		<axis xyz="0 1 0"/>
+		<limit effort="1" lower="-0.19" upper="0" velocity="1"/>
+		<origin xyz="${((base_l-arm_l)/2) + 0.028} ${-(base_w+arm_w)/2} ${(arm_h-base_h)/2}"/>
+	</joint>
+	<joint name ="arm_to_mount" type="fixed">
+		<parent link="arm"/>
+		<child link="mount"/>
+		<origin xyz="${(arm_l+mount_l)/2} 0.02 0"/>
+	</joint>
+	<joint name ="mount_to_end_effector_1" type="revolute">
+		<parent link="mount"/>
+		<child link="end_effector_1"/>
+		<axis xyz="0 1 0"/>
+		<limit effort="1" lower="0" upper="1.58" velocity="1"/>
+		<origin xyz="${(mount_l+end_effector_1_l)/2} 0.012 0.008"/>
+	</joint>
+	<joint name ="end_effector_1_to_end_effector_2" type="fixed">
+		<parent link="end_effector_1"/>
+		<child link="end_effector_2"/>
+		<origin xyz="${(end_effector_1_l-end_effector_2_l)/2} 0 ${(end_effector_2_h-end_effector_1_h)/2}"/>
+	</joint>
 </robot>

File: catkin_ws/src/me212arm/model/my_robot.xacro (robot description, xacro)
@@ -17,10 +17,10 @@
 <xacro:property name="end_effector_2_h" value="0.08"/>
 <xacro:property name="pi" value="3.141592654"/>
-	<link name="base">   <!-- need to change x to y, y to -x -->
+	<link name="base">
 		<visual>
 			<geometry>
 				<box size="${base_l} ${base_w} ${base_h}"/>
 			</geometry>
-			<origin rpy="0 0 0" xyz="0 0 0"/> <!-- CHANGE LATER -->
+			<origin rpy="0 0 0" xyz="0 0 0"/>
 		</visual>
 	</link>
@@ -30,5 +30,5 @@
 				<box size="${arm_l} ${arm_w} ${arm_h}"/>
 			</geometry>
-			<origin rpy="0 0 0" xyz="${(arm_length-base_length)/2} "/>
+			<origin rpy="0 0 0" xyz="${(arm_l-base_l)/2} "/>
 		</visual>
 	</link>

Commit message: working arm xacro/urdf file

File: catkin_ws/src/me212arm/model/me212arm.xacro (robot description, xacro)
@@ -1,83 +1,69 @@
 <?xml version="1.0"?>
-<robot xmlns:xacro="http://www.ros.org/wiki/xacro" name="my_robot">
-<xacro:property name="base_l" value="0.07"/>
-<xacro:property name="base_w" value="0.06"/>
-<xacro:property name="base_h" value="0.04"/>
-<xacro:property name="arm_l" value="0.26"/>
-<xacro:property name="arm_w" value="0.01"/>
-<xacro:property name="arm_h" value="0.01"/>
-<xacro:property name="mount_l" value="0.50"/>
-<xacro:property name="mount_w" value="0.061"/>
-<xacro:property name="mount_h" value="0.07"/>
-<xacro:property name="end_effector_1_l" value="0.207"/>
-<xacro:property name="end_effector_1_w" value="0.01"/>
-<xacro:property name="end_effector_1_h" value="0.01"/>
-<xacro:property name="end_effector_2_l" value="0.01"/>
-<xacro:property name="end_effector_2_w" value="0.01"/>
-<xacro:property name="end_effector_2_h" value="0.08"/>
-<xacro:property name="pi" value="3.141592654"/>
-	<link name="base">
-		<visual>
-			<geometry>
-				<box size="${base_l} ${base_w} ${base_h}"/>
-			</geometry>
-			<origin rpy="0 0 0" xyz="0 0 0"/>
-		</visual>
-	</link>
-	<link name="arm">
-		<visual>
-			<geometry>
-				<box size="${arm_l} ${arm_w} ${arm_h}"/>
-			</geometry>
-			<origin rpy="0 0 0" xyz="${(arm_l-base_l)/2} "/>
-		</visual>
-	</link>
-	<link name="mount">
-		<visual>
-			<geometry>
-				<box size="${mount_l} ${mount_w} ${mount_h}"/>
-			</geometry>
-			<origin xyz=""/>
-		</visual>
-	</link>
-	<link name="end_effector_1">
-		<visual>
-			<geometry>
-				<box size="${end_effector_1_l} ${end_effector_1_w} ${end_effector_1_h}"/>
-			</geometry>
-			<origin xyz=""/>
-		</visual>
-	</link>
-	<link name="end_effector_2">
-		<visual>
-			<geometry>
-				<box size="${end_effector_2_l} ${end_effector_2_w} ${end_effector_2_h}"/>
-			</geometry>
-			<origin xyz=""/>
-		</visual>
-	</link>
-	<joint name ="base_to_arm" type="prismatic">
-		<parent link="base"/>
-		<child link="arm"/>
-		<axis xyz="0 1 0"/>
-		<limit effort="1" lower="-0.19" upper="0" velocity="1"/>
-		<origin xyz="${((base_l-arm_l)/2) + 0.028} ${-(base_w+arm_w)/2} ${(arm_h-base_h)/2}"/>
-	</joint>
-	<joint name ="arm_to_mount" type="fixed">
-		<parent link="arm"/>
-		<child link="mount"/>
-		<origin xyz="${(arm_l+mount_l)/2} 0.02 0"/>
-	</joint>
-	<joint name ="mount_to_end_effector_1" type="revolute">
-		<parent link="mount"/>
-		<child link="end_effector_1"/>
-		<axis xyz="0 1 0"/>
-		<limit effort="1" lower="0" upper="1.58" velocity="1"/>
-		<origin xyz="${(mount_l+end_effector_1_l)/2} 0.012 0.008"/>
-	</joint>
-	<joint name ="end_effector_1_to_end_effector_2" type="fixed">
-		<parent link="end_effector_1"/>
-		<child link="end_effector_2"/>
-		<origin xyz="${(end_effector_1_l-end_effector_2_l)/2} 0 ${(end_effector_2_h-end_effector_1_h)/2}"/>
-	</joint>
+<robot xmlns:xacro="http://www.ros.org/wiki/xacro" name="me212bot">
+<xacro:property name="link1_length" value="0.1778" />
+<xacro:property name="link2_length" value="0.235" />
+<xacro:property name="M_PI" value="3.1415926" />
+<link name="arm_base">
+    <visual>
+        <geometry>
+            <box size="0.01 0.01 0.05" />
+        </geometry>
+        <origin rpy="0 0 0" xyz="0 0 0"/>
+        <material name="color1">
+            <color rgba="0.5 0.5 0.0 1"/>
+        </material>
+    </visual>
+</link>
+<link name="link1">
+    <visual>
+        <geometry>
+            <box size="0.01 0.01 ${link1_length}" />
+        </geometry>
+        <origin rpy="0 0 0" xyz="0 0 ${link1_length/2}"/>
+        <material name="color2">
+            <color rgba="0.5 0.0 0.5 1"/>
+        </material>
+    </visual>
+</link>
+<link name="link2">
+    <visual>
+        <geometry>
+            <box size="0.01 0.01 ${link2_length}" />
+        </geometry>
+        <origin rpy="0 0 0" xyz="0 0 ${link2_length/2}"/>
+        <material name="color3">
+            <color rgba="0.0 0.5 0.5 1"/>
+        </material>
+    </visual>
+</link>
+<link name="tcp">
+    <visual>
+        <geometry>
+            <sphere radius="0.01" />
+        </geometry>
+        <origin rpy="0 0 0" xyz="0 0 0"/>
+        <material name="color4">
+            <color rgba="0.5 0.5 0.5 1"/>
+        </material>
+    </visual>
+</link>
+<joint name="joint1" type="revolute">
+    <parent link="arm_base"/>
+    <child link="link1"/>
+    <origin xyz="0 0 0" />
+    <limit effort="300" lower="${-M_PI}" upper="${M_PI}" velocity="7.33"/>
+    <axis xyz="0 -1 0"/>
+</joint>
+<joint name="joint2" type="revolute">
+    <parent link="link1"/>
+    <child link="link2"/>
+    <origin xyz="0 0 ${link1_length}" />
+    <limit effort="300" lower="${-M_PI}" upper="${M_PI}" velocity="7.33"/>
+    <axis xyz="0 -1 0"/>
+</joint>
+<joint name="joint3" type="fixed">
+    <parent link="link2"/>
+    <child link="tcp"/>
+    <origin xyz="0 0 ${link2_length}" />
+</joint>
 </robot>

File: catkin_ws/src/me212arm/model/me212armtest.xacro (robot description, xacro)
@@ -7,5 +7,5 @@
 <xacro:property name="arm_w" value="0.01"/>
 <xacro:property name="arm_h" value="0.01"/>
-<xacro:property name="mount_l" value="0.050"/>
+<xacro:property name="mount_l" value="0.50"/>
 <xacro:property name="mount_w" value="0.061"/>
 <xacro:property name="mount_h" value="0.07"/>
@@ -30,5 +30,5 @@
 				<box size="${arm_l} ${arm_w} ${arm_h}"/>
 			</geometry>
-			<origin rpy="0 0 0" xyz="0 0 0"/>
+			<origin rpy="0 0 0" xyz="${(arm_l-base_l)/2} "/>
 		</visual>
 	</link>
@@ -38,5 +38,5 @@
 				<box size="${mount_l} ${mount_w} ${mount_h}"/>
 			</geometry>
-			<origin xyz="0 0 0"/>
+			<origin xyz=""/>
 		</visual>
 	</link>
@@ -46,5 +46,5 @@
 				<box size="${end_effector_1_l} ${end_effector_1_w} ${end_effector_1_h}"/>
 			</geometry>
-			<origin xyz="0 0 0"/>
+			<origin xyz=""/>
 		</visual>
 	</link>
@@ -54,5 +54,5 @@
 				<box size="${end_effector_2_l} ${end_effector_2_w} ${end_effector_2_h}"/>
 			</geometry>
-			<origin xyz="0 0 0"/>
+			<origin xyz=""/>
 		</visual>
 	</link>
@@ -60,6 +60,6 @@
 		<parent link="base"/>
 		<child link="arm"/>
-		<axis xyz="1 0 0"/>
-		<limit effort="1" lower="0" upper="0.16" velocity="1"/>
+		<axis xyz="0 1 0"/>
+		<limit effort="1" lower="-0.19" upper="0" velocity="1"/>
 		<origin xyz="${((base_l-arm_l)/2) + 0.028} ${-(base_w+arm_w)/2} ${(arm_h-base_h)/2}"/>
 	</joint>
@@ -72,7 +72,7 @@
 		<parent link="mount"/>
 		<child link="end_effector_1"/>
-		<axis xyz="1 0 0"/>
-		<limit effort="1" lower="-1.58" upper="0" velocity="1"/>
-		<origin xyz="${(mount_l+end_effector_1_l)/2} 0.012 -0.008"/>
+		<axis xyz="0 1 0"/>
+		<limit effort="1" lower="0" upper="1.58" velocity="1"/>
+		<origin xyz="${(mount_l+end_effector_1_l)/2} 0.012 0.008"/>
 	</joint>
 	<joint name ="end_effector_1_to_end_effector_2" type="fixed">
