Commit message: played with urdf files on the whole robot assembly

File: catkin_ws/src/me212arm/model/my_robot.urdf (robot description, URDF)
Before this commit: robot my_robot, 5 links, 4 joints
Joints:
- joint base_to_arm: limit lower=0 upper=0.19 effort=1 velocity=1 -> lower=0 upper=0.16 effort=1 velocity=1
- joint mount_to_end_effector_1: origin xyz=0.1285 0.012 0.008 -> xyz=0.1285 0.012 -0.008
