Commit message: created assembly file

File: catkin_ws/src/me212bot/model/my_assembly.xacro (robot description, xacro)
@@ -6,5 +6,5 @@
         <parent link="robot_base"/>
         <child link="base"/>
-        <origin xyz="0.05 0.05 0.30" />
+        <origin xyz="0.121 -0.095 0.30" />
     </joint>
 </robot>
